Commit message: update kinematics for a tcp joint

File: code/urdf/ur5e/ur5e_onrobot.urdf (robot description, URDF)
Before this commit: robot rilab_robot, 16 links, 15 joints
Joints:
- joint gripper_tcp_joint: origin xyz=0 0. 0.17 rpy=0 0 0 -> xyz=0 0. 0.185 rpy=0 0 0

Commit message: update camera joint

File: code/urdf/ur5e/ur5e_onrobot.urdf (robot description, URDF)
Before this commit: robot rilab_robot, 16 links, 15 joints
Links:
- removed link tool0
- added link camera_base_link, mass 0.199035856566616
- added link mount_link, mass 0.1879; collision mesh filename=package://ir_gazebo/urdf/ur5e/meshes/collision/mount.stl scale=0.0001 0.0001 0.0001; visual mesh filename=package://ir_gazebo/urdf/ur5e/meshes/collision/mount.stl scale=0.0001 0.0001 0.0001
Joints:
- removed joint ee_fixed_joint
- added joint mount_camera_joint: type fixed, parent mount_link, child camera_base_link, origin xyz=0 0. 0.093 rpy=0 0 0, axis 0 1 0
- added joint mount_joint: type fixed, parent wrist_3_link, child mount_link, origin xyz=0.0 0.045 0.0 rpy=0 3.141592 3.141592, axis 0 1 0
- joint gripper_base_joint: origin xyz=0 0. 0. rpy=-1.57 0 0 -> xyz=0 0.1 0. rpy=-1.57 0 0; parent tool0 -> wrist_3_link

Commit message: update self-collison checker

File: code/urdf/ur5e/ur5e_onrobot.urdf (robot description, URDF)
Before this commit: robot rilab_robot, 17 links, 16 joints
Joints:
- joint mount_camera_joint: origin xyz=0 0. 0.093 rpy=0 0 0 -> xyz=0 -0.015 0.093 rpy=0 0 0

Commit message: update UR5e-onrobot-realsense configuration

File: code/urdf/ur5e/ur5e_onrobot.urdf (robot description, URDF)
Before this commit: robot rilab_robot, 17 links, 16 joints
Joints:
- joint mount_joint: origin xyz=0.0 0.045 0.0 rpy=0 3.141592 3.141592 -> xyz=0.0 0.09 0.0 rpy=0 3.141592 3.141592

Commit message: update collision checker

File: code/urdf/ur5e/ur5e_onrobot.urdf (robot description, URDF)
Before this commit: robot rilab_robot, 17 links, 16 joints
Links:
- link camera_base_link: geometry visual mesh filename=package://ir_gazebo/urdf/realsense_d435/meshes/visual/d435.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 scale=0.001 0.001 0.001
Joints:
- joint mount_camera_joint: origin xyz=0 -0.015 0.093 rpy=0 0 0 -> xyz=0 -0.015 0.093 rpy=0 1.57 0
