Commit message: update ril_robot ver.

File: code/urdf/ur5e/ril_robot.urdf (robot description, URDF)
Before this commit: robot rilab_robot, 17 links, 16 joints
Links:
- link base_link: geometry collision mesh filename=package://ril_manipulator/urdf/ur5e/meshes/collision/base.s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; visual mesh filename=package://ril_manipulator/urdf/ur5e/meshes/visual/base.dae
- link camera_base_link: geometry visual mesh filename=package://ir_gazebo/urdf/realsense_d435/meshes/visual/d435.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
- link forearm_link: geometry collision mesh filename=package://ril_manipulator/urdf/ur5e/meshes/collision/forear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; visual mesh filename=package://ril_manipulator/urdf/ur5e/meshes/visual/forearm.d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
- link gripper_base_link: geometry collision mesh filename=package://ril_manipulator/urdf/rg2/meshes/collision/gripper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; visual mesh filename=package://ril_manipulator/urdf/rg2/meshes/visual/gripper_ba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
- link gripper_finger1_finger_link: geometry collision mesh filename=package://ril_manipulator/urdf/rg2/meshes/collision/gripper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; visual mesh filename=package://ril_manipulator/urdf/rg2/meshes/visual/gripper_fi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
- link gripper_finger1_finger_tip_link: geometry collision mesh filename=package://ril_manipulator/urdf/rg2/meshes/collision/gripper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; visual mesh filename=package://ril_manipulator/urdf/rg2/meshes/visual/gripper_fi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
- link gripper_finger1_inner_knuckle_link: geometry collision mesh filename=package://ril_manipulator/urdf/rg2/meshes/collision/gripper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; visual mesh filename=package://ril_manipulator/urdf/rg2/meshes/visual/gripper_fi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
- link gripper_finger2_finger_link: geometry collision mesh filename=package://ril_manipulator/urdf/rg2/meshes/collision/gripper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; visual mesh filename=package://ril_manipulator/urdf/rg2/meshes/visual/gripper_fi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
- link gripper_finger2_finger_tip_link: geometry collision mesh filename=package://ril_manipulator/urdf/rg2/meshes/collision/gripper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; visual mesh filename=package://ril_manipulator/urdf/rg2/meshes/visual/gripper_fi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
- link gripper_finger2_inner_knuckle_link: geometry collision mesh filename=package://ril_manipulator/urdf/rg2/meshes/collision/gripper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; visual mesh filename=package://ril_manipulator/urdf/rg2/meshes/visual/gripper_fi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
- link mount_link: geometry collision mesh filename=package://ril_manipulator/urdf/ur5e/meshes/collision/mount.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 scale=0.0001 0.0001 0.0001; visual mesh filename=package://ril_manipulator/urdf/ur5e/meshes/collision/mount.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 scale=0.0001 0.0001 0.0001
- link shoulder_link: geometry collision mesh filename=package://ril_manipulator/urdf/ur5e/meshes/collision/should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; visual mesh filename=package://ril_manipulator/urdf/ur5e/meshes/visual/shoulder.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
- link upper_arm_link: geometry collision mesh filename=package://ril_manipulator/urdf/ur5e/meshes/collision/uppera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; visual mesh filename=package://ril_manipulator/urdf/ur5e/meshes/visual/upperarm.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
- link wrist_1_link: geometry collision mesh filename=package://ril_manipulator/urdf/ur5e/meshes/collision/wrist1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; visual mesh filename=package://ril_manipulator/urdf/ur5e/meshes/visual/wrist1.dae
- link wrist_2_link: geometry collision mesh filename=package://ril_manipulator/urdf/ur5e/meshes/collision/wrist2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; visual mesh filename=package://ril_manipulator/urdf/ur5e/meshes/visual/wrist2.dae
- link wrist_3_link: geometry collision mesh filename=package://ril_manipulator/urdf/ur5e/meshes/collision/wrist3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; visual mesh filename=package://ril_manipulator/urdf/ur5e/meshes/visual/wrist3.dae
Joints:
- joint gripper_base_joint: origin xyz=0 0.1 0. rpy=-1.57 0 0 -> xyz=0 0.1 0. rpy=-1.57 -1.57  0
- joint mount_camera_joint: axis 0 1 0 -> (none); origin xyz=0 -0.015 0.093 rpy=0 0 0 -> xyz=0. -0.025 0.087 rpy=1.5707963267948966 0 0
- joint mount_joint: origin xyz=0.0 0.09 0.0 rpy=0 3.141592 3.141592 -> xyz=0.0 0.09 0.0 rpy=3.14 -1.57 0
- joint wrist_3_joint: limit lower=-3.14159265359 upper=3.14159265359 effort=28.0 velocity=6.28 -> lower=-3.141592653589793 upper=3.141592653589793 effort=28.0 velocity=6.28

Commit message: update kinematics config

File: code/urdf/ur5e/ril_robot.urdf (robot description, URDF)
Before this commit: robot rilab_robot, 17 links, 16 joints
Joints:
- joint gripper_base_joint: origin xyz=0 0.1 0. rpy=-1.57 -1.57  0 -> xyz=0 0.1 0. rpy=-1.57 0 0
- joint mount_joint: origin xyz=0.0 0.09 0.0 rpy=3.14 -1.57 0 -> xyz=0.0 0.09 0.0 rpy=3.14 0 0

Commit message: update

File: code/urdf/ur5e/ril_robot.urdf (robot description, URDF)
Before this commit: robot rilab_robot, 17 links, 16 joints
Links:
- link camera_base_link: geometry visual mesh filename=package://ril_manipulator/urdf/realsense_d435/meshes/visual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
